Commit message: Several fixes.

File: urdf/apriltag_bottle.xacro (robot description, xacro)
@@ -16,4 +16,5 @@
        (C) 2018 fnh, hendrich@informatik.uni-hamburg.de
        Usage:
+       <xacro:include filename="$(find tiago_world)/urdf/materials.xacro" />
        <xacro:apriltag_bottle
               namespace="" name="bitter_orange_bottle" weight="1.0"
@@ -21,12 +22,8 @@
               tagFamily="36h11" tagID="201" tagSize="0.06" />
    -->
-  <xacro:include filename="$(find thiago_world)/urdf/materials.xacro" />
-  <xacro:include filename="$(find thiago_world)/urdf/bottle.xacro" />
+  <xacro:include filename="$(find tiago_world)/urdf/bottle.xacro" />
   <xacro:include filename="$(find tams_apriltags)/urdf/apriltag_marker.xacro" />
   <xacro:macro name="apriltag_bottle"
                params="namespace name weight rvizMaterial gazeboMaterial tagFamily tagID tagSize " >
-    <!-- main bottle body -->
-    <xacro:bottle namespace="${namespace}" name="${name}"
-                  rvizMaterial="${rvizMaterial}" gazeboMaterial="${gazeboMaterial}" />
     <!-- apriltag on the front of the bottle -->
     <link name="${namespace}${name}_atag_link">
@@ -52,8 +49,11 @@
       <kd>1.0</kd>
     </gazebo>
+    <!-- main bottle body -->
+    <xacro:bottle namespace="${namespace}" name="${name}" weight="${weight}"
+                  rvizMaterial="${rvizMaterial}" gazeboMaterial="${gazeboMaterial}" />
     <joint name="${namespace}${name}_atag_joint" type="fixed">
       <parent link="${namespace}${name}" />
       <child link="${namespace}${name}_atag_link" />
-      <origin xyz="0.04 0 ${0.25-tagSize}" rpy="0 0 0" />
+      <origin xyz="0.04 0 ${0.25-tagSize}" rpy="0 1.571 0" />
     </joint>
   </xacro:macro>

File: urdf/bar_counter.xacro (robot description, xacro)
@@ -13,5 +13,5 @@
        <xacro:bar_counter name="counter" />
    -->
-  <xacro:include filename="$(find thiago_world)/urdf/materials.xacro" />
+  <xacro:include filename="$(find tiago_world)/urdf/materials.xacro" />
   <xacro:macro name="bar_counter"
                params="name" >
@@ -26,5 +26,5 @@
         <origin xyz="0 0 0" rpy="0 0 0" />
         <geometry>
-          <mesh filename="file://$(find thiago_world)/meshes/bartresen_binary.stl" scale="0.001 0.001 0.001" />
+          <mesh filename="file://$(find tiago_world)/meshes/bartresen_binary.stl" scale="0.001 0.001 0.001" />
         </geometry>
       </collision>
@@ -32,5 +32,5 @@
         <origin xyz="0 0 0" rpy="0 0 0" />
         <geometry>
-          <mesh filename="file://$(find thiago_world)/meshes/bartresen_binary.stl" scale="0.001 0.001 0.001" />
+          <mesh filename="file://$(find tiago_world)/meshes/bartresen_binary.stl" scale="0.001 0.001 0.001" />
         </geometry>
         <material name="noyer_wood" >
@@ -41,5 +41,5 @@
     <gazebo reference="${name}">
       <!-- material/texture definition for Gazebo -->
-      <material>thiago/Wood</material> -->
+      <material>tiago/Wood</material> -->
       <turnGravityOff>false</turnGravityOff>
       <selfCollide>false</selfCollide>

File: urdf/bar_stool.xacro (robot description, xacro)
@@ -13,5 +13,5 @@
        <xacro:bar_stool name="stool_1" />
    -->
-  <xacro:include filename="$(find thiago_world)/urdf/materials.xacro" />
+  <xacro:include filename="$(find tiago_world)/urdf/materials.xacro" />
   <xacro:macro name="bar_stool" params="name" >
     <!-- main body with mesh collision and visual model -->
@@ -25,5 +25,5 @@
         <origin xyz="0 0 0" rpy="0 0 0" />
         <geometry>
-          <mesh filename="file://$(find thiago_world)/meshes/bar_stool_binary.stl" scale="0.001 0.001 0.001" />
+          <mesh filename="file://$(find tiago_world)/meshes/bar_stool_binary.stl" scale="0.001 0.001 0.001" />
         </geometry>
       </collision>
@@ -31,5 +31,5 @@
         <origin xyz="0 0 0" rpy="0 0 0" />
         <geometry>
-          <mesh filename="file://$(find thiago_world)/meshes/bar_stool_binary.stl" scale="0.001 0.001 0.001" />
+          <mesh filename="file://$(find tiago_world)/meshes/bar_stool_binary.stl" scale="0.001 0.001 0.001" />
         </geometry>
         <material name="silver" >
@@ -40,5 +40,5 @@
     <gazebo reference="${name}">
       <!-- material/texture definition for Gazebo -->
-      <material>thiago/Silver</material> -->
+      <material>tiago/Silver</material> -->
       <turnGravityOff>false</turnGravityOff>
       <selfCollide>false</selfCollide>

File: urdf/bottle.xacro (robot description, xacro)
@@ -11,10 +11,9 @@
        (C) 2018 fnh, hendrich@informatik.uni-hamburg.de
        Usage:
-       <xacro:apriltag_bottle
-              namespace="" name="bitter_orange_bottle" weight="1.0"
-              rvizMaterial="orange" gazeboMaterial="Gazebo/Orange"
-              tagFamily="36h11" tagID="201" tagSize="0.06" />
+       <xacro:include filename="$(find tiago_world)/urdf/materials.xacro" />
+       <xacro:bottle
+              namespace="" name="bitter_lemon_bottle" weight="1.0"
+              rvizMaterial="orange" gazeboMaterial="Gazebo/Orange" />
    -->
-  <xacro:include filename="$(find thiago_world)/urdf/materials.xacro" />
   <xacro:macro name="bottle"
                params="namespace name weight rvizMaterial gazeboMaterial" >
@@ -32,5 +31,5 @@
         <origin xyz="0 0 ${0.5*0.25}" rpy="0 0 0" />
         <geometry>
-          <cylinder radius="0.04" height="0.3" />
+          <cylinder radius="0.04" length="0.3" />
         </geometry>
       </collision>
@@ -38,5 +37,5 @@
         <origin xyz="0 0 0" rpy="0 0 0" />
         <geometry>
-          <mesh filename="file://$(find thiago_world)/meshes/bottle_binary.stl" scale="1 1 1" />
+          <mesh filename="file://$(find tiago_world)/meshes/bottle_binary.stl" scale="0.001 0.001 0.001" />
         </geometry>
         <material name="${rvizMaterial}" >

File: urdf/bottle_demo.xacro (robot description, xacro)
@@ -4,15 +4,15 @@
        xmlns:interface="http://playerstage.sourceforge.net/gazebo/xmlschema/#interface"
        xmlns:xacro="http://www.ros.org/wiki/xacro"
-       name="apriltag_demo">
-  <xacro:include filename="$(find thiago_world)/urdf/materials.xacro" />
-  <xacro:include filename="$(find thiago_world)/urdf/bottle.xacro" />
-  <xacro:include filename="$(find thiago_world)/urdf/apriltag_bottle.xacro" />
-  <xacro:include filename="$(find thiago_world)/urdf/easy_grasp_bottle.xacro" />
-  <xacro:include filename="$(find thiago_world)/urdf/ikea_glass.xacro" />
+       name="bottle_demo">
+  <xacro:include filename="$(find tiago_world)/urdf/materials.xacro" />
+  <xacro:include filename="$(find tiago_world)/urdf/bottle.xacro" />
+  <xacro:include filename="$(find tiago_world)/urdf/apriltag_bottle.xacro" />
+  <xacro:include filename="$(find tiago_world)/urdf/easy_grasp_bottle.xacro" />
+  <xacro:include filename="$(find tiago_world)/urdf/ikea_glass.xacro" />
   <link name="world" />
-  <link name="thiago/world" />
+  <link name="tiago/world" />
   <joint name="hugo" type="fixed">
     <parent link="world" />
-    <child  link="thiago/world" />
+    <child  link="tiago/world" />
   </joint>
   <xacro:bottle
@@ -24,28 +24,28 @@
   <xacro:apriltag_bottle
          namespace="" name="apriltag_bottle_213" weight="0.5"
-         rvizMaterial="green" gazeboMaterial="Gazebo/Green"
+         rvizMaterial="blue" gazeboMaterial=""
          tagFamily="36h11" tagID="213" tagSize="0.06" />
   <xacro:ikea_glass
-         namespace="" name="ikea_glass_1" weight="0.5"
-         rvizMaterial="grey" gazeboMaterial="Gazebo/Grey" />
+         namespace="" name="ikea_glass_1" liquid_weight="0.5"
+         rvizMaterial="yellow" gazeboMaterial="Gazebo/Yellow" />
   <joint name="green_bottle_joint" type="fixed">
     <parent link="world" />
     <child  link="green_bottle" />
-    <origin xyz="1 0 0" rpy="0 1.571 0" />
+    <origin xyz="1 0 0.001" rpy="0 0 0" />
   </joint>
   <joint name="bitter_orange_bottle_joint" type="fixed">
     <parent link="world" />
     <child  link="bitter_orange_bottle" />
-    <origin xyz="1 0.2 0" rpy="0 1.571 0" />
+    <origin xyz="1 0.2 0.001" rpy="0 0 0" />
   </joint>
   <joint name="apriltag_bottle_213_joint" type="fixed">
     <parent link="world" />
     <child  link="apriltag_bottle_213" />
-    <origin xyz="1 0.4 0" rpy="0 1.571 0" />
+    <origin xyz="1 0.4 0.001" rpy="0 0 0" />
   </joint>
   <joint name="ikea_glass_joint" type="fixed">
     <parent link="world" />
     <child  link="ikea_glass_1" />
-    <origin xyz="1 0.4 0" rpy="0 1.571 0" />
+    <origin xyz="1 0.6 0.002" rpy="0 0 0" />
   </joint>
 </robot>

File: urdf/easy_grasp_bottle.xacro (robot description, xacro)
@@ -13,11 +13,11 @@
        (C) 2018 fnh, hendrich@informatik.uni-hamburg.de
        Usage:
-       <xacro:apriltag_bottle
-              namespace="" name="bitter_orange_bottle" weight="1.0"
+       <xacro:include filename="$(find tiago_world)/urdf/materials.xacro" />
+       <xacro:easy_grasp_bottle
+              namespace="" name="easy_grasp__bottle" weight="1.0"
               rvizMaterial="orange" gazeboMaterial="Gazebo/Orange"
               tagFamily="36h11" tagID="201" tagSize="0.06" />
    -->
-  <xacro:include filename="$(find thiago_world)/urdf/materials.xacro" />
-  <xacro:macro name="bottle"
+  <xacro:macro name="easy_grasp_bottle"
                params="namespace name weight rvizMaterial gazeboMaterial" >
     <!-- main body with cylinder collision model and bottle mesh for visual -->
@@ -34,5 +34,5 @@
         <origin xyz="0 0 ${0.5*0.25}" rpy="0 0 0" />
         <geometry>
-          <cylinder radius="0.04" height="0.3" />
+          <cylinder radius="0.04" length="0.3" />
         </geometry>
       </collision>
@@ -40,5 +40,5 @@
         <origin xyz="0 0 0" rpy="0 0 0" />
         <geometry>
-          <mesh filename="file://$(find thiago_world)/meshes/bottle_easy_grasp_binary.stl" scale="1 1 1" />
+          <mesh filename="file://$(find tiago_world)/meshes/easy_grasp_bottle_binary.stl" scale="0.001 0.001 0.001" />
         </geometry>
         <material name="${rvizMaterial}" >

File: urdf/ikea_glass.xacro (robot description, xacro)
@@ -11,9 +11,9 @@
        (C) 2018 fnh, hendrich@informatik.uni-hamburg.de
        Usage:
+       <xacro:include filename="$(find tiago_world)/urdf/materials.xacro" />
        <xacro:ikea_glass
-              namespace="" name="bitter_orange_bottle" weight="0.2"
-              rvizMaterial="orange" gazeboMaterial="Gazebo/Orange" />
+              namespace="" name="ikea_glass_1" weight="0.2"
+              rvizMaterial="white" gazeboMaterial="Gazebo/White" />
    -->
-  <xacro:include filename="$(find thiago_world)/urdf/materials.xacro" />
   <xacro:macro name="ikea_glass"
                params="namespace name liquid_weight rvizMaterial gazeboMaterial" >
@@ -32,5 +32,5 @@
         <origin xyz="0 0 0" rpy="0 0 0" />
         <geometry>
-          <mesh filename="file://$(find thiago_world)/meshes/ikea_glass_binary.stl" scale="1 1 1" />
+          <mesh filename="file://$(find tiago_world)/meshes/ikea_glass_binary.stl" scale="0.001 0.001 0.001" />
         </geometry>
       </collision>
@@ -38,5 +38,5 @@
         <origin xyz="0 0 0" rpy="0 0 0" />
         <geometry>
-          <mesh filename="file://$(find thiago_world)/meshes/ikea_glass_binary.stl" scale="1 1 1" />
+          <mesh filename="file://$(find tiago_world)/meshes/ikea_glass_binary.stl" scale="0.001 0.001 0.001" />
         </geometry>
         <material name="${rvizMaterial}" >

File: urdf/thiago_command_card.xacro (robot description, xacro)
@@ -4,6 +4,6 @@
        xmlns:interface="http://playerstage.sourceforge.net/gazebo/xmlschema/#interface"
        xmlns:xacro="http://www.ros.org/wiki/xacro"
-       name="thiago_card">
-  <!-- ROS xacro/urdf model of one "Thiago demo command card",
+       name="tiago_card">
+  <!-- ROS xacro/urdf model of one "Tiago demo command card",
        which has a command/cocktail recipe on the front and an
        apriltag marker on the back.
@@ -13,5 +13,5 @@
        (C) 2018 fnh, hendrich@informatik.uni-hamburg.de
        Usage:
-       <xacro:thiago_command_card namespace="" name="thiago_reset_card" front="reset.png"
+       <xacro:tiago_command_card namespace="" name="tiago_reset_card" front="reset.png"
               family="36h11" tagID="201" dx="0.1" dy="0.06" dz="0.005"/>
        <xacro:apriltag_marker namespace="doro/" name="apriltag13" parent="base_link"
@@ -21,5 +21,5 @@
    -->
   <xacro:include filename="$(find tams_apriltags)/urdf/apriltag_marker.xacro" />
-  <xacro:macro name="thiago_command_card" params="namespace name texture gazeboMaterial family tagID tagSize dx dy dz" >
+  <xacro:macro name="tiago_command_card" params="namespace name texture gazeboMaterial family tagID tagSize dx dy dz" >
     <!-- main body with collision but without visual -->
     <link name="${namespace}${name}">
@@ -40,5 +40,5 @@
           <box size="${dx} ${dy} ${dz}" />
         </geometry>
-        <material name="thiago_command_card_white/${name}">
+        <material name="tiago_command_card_white/${name}">
           <color rgba="1.0 1.0 1.0 1.0"/>
         </material>
@@ -64,5 +64,5 @@
         </geometry>
         <!-- material definition for rviz -->
-        <material name="thiago_command_card_texture/${name}/texture" >
+        <material name="tiago_command_card_texture/${name}/texture" >
           <texture filename="file://$(find tams_apriltags)/Media/materials/textures/${texture}" />
         </material>
