Commit message: Get bar_demo to launch.

File: urdf/bar_cupboard.xacro (robot description, xacro)
@@ -4,7 +4,7 @@
        xmlns:interface="http://playerstage.sourceforge.net/gazebo/xmlschema/#interface"
        xmlns:xacro="http://www.ros.org/wiki/xacro"
-       name="bar_counter">
-  <!-- ROS xacro/urdf model of a bar counter ("Tresen") with wood
-       texture and some shelves on the back (robot) side.
+       name="bar_cupboard">
+  <!-- ROS xacro/urdf model of a bar shelf/cupboard with wood
+       texture.
        Origin is at the bottom, centered in x and y.
        2018.05.17 - created
@@ -12,12 +12,12 @@
        Usage:
        <xacro:include filename="$(find tiago_world)/urdf/materials.xacro" />
-       <xacro:bar_counter name="counter" />
+       <xacro:bar_cupboard name="cupboard" />
    -->
-  <xacro:macro name="bar_counter"
+  <xacro:macro name="bar_cupboard"
                params="name" >
     <!-- main body with mesh collision and visual model -->
     <link name="${name}">
       <inertial>
-        <mass value="200" />
+        <mass value="300" />
         <origin xyz="0 0 0" rpy="0 0 0" />
         <inertia ixx="0.01" ixy="0" ixz="0" iyy="0.01" iyz="0" izz="0.01" />
@@ -26,5 +26,5 @@
         <origin xyz="0 0 0" rpy="0 0 0" />
         <geometry>
-          <mesh filename="file://$(find tiago_world)/meshes/bartresen_binary.stl" scale="0.001 0.001 0.001" />
+          <mesh filename="file://$(find tiago_world)/meshes/cupboard_binary.stl" scale="0.001 0.001 0.001" />
         </geometry>
       </collision>
@@ -32,5 +32,5 @@
         <origin xyz="0 0 0" rpy="0 0 0" />
         <geometry>
-          <mesh filename="file://$(find tiago_world)/meshes/bartresen_binary.stl" scale="0.001 0.001 0.001" />
+          <mesh filename="file://$(find tiago_world)/meshes/cupboard_binary.stl" scale="0.001 0.001 0.001" />
         </geometry>
         <material name="noyer_wood" >

File: urdf/bar_stool.xacro (robot description, xacro)
@@ -11,7 +11,7 @@
        (C) 2018 fnh, hendrich@informatik.uni-hamburg.de
        Usage:
+       <xacro:include filename="$(find tiago_world)/urdf/materials.xacro" />
        <xacro:bar_stool name="stool_1" />
    -->
-  <xacro:include filename="$(find tiago_world)/urdf/materials.xacro" />
   <xacro:macro name="bar_stool" params="name" >
     <!-- main body with mesh collision and visual model -->
@@ -33,6 +33,6 @@
           <mesh filename="file://$(find tiago_world)/meshes/bar_stool_binary.stl" scale="0.001 0.001 0.001" />
         </geometry>
-        <material name="silver" >
-          <!-- <color rgba="1.0 1.0 1.0 1.0"/> -->
+        <material name="${name}_bar_stool_gray" >
+          <color rgba="0.7 0.4 0.4 1.0" />
         </material>
       </visual>
@@ -40,5 +40,5 @@
     <gazebo reference="${name}">
       <!-- material/texture definition for Gazebo -->
-      <material>tiago/Silver</material> -->
+      <material>tiago/Coke</material>
       <turnGravityOff>false</turnGravityOff>
       <selfCollide>false</selfCollide>
