Commit message: Add spawn_xacro launch. Move tiago_command_card here.

File: urdf/bottle.xacro (robot description, xacro)
@@ -29,7 +29,7 @@
       <collision>
         <!-- Schweppes 1-liter plastic bottle -->
-        <origin xyz="0 0 ${0.5*0.25}" rpy="0 0 0" />
+        <origin xyz="0 0 ${0.5*0.284}" rpy="0 0 0" />
         <geometry>
-          <cylinder radius="0.04" length="0.3" />
+          <cylinder radius="0.04" length="0.284" />
         </geometry>
       </collision>
@@ -55,9 +55,9 @@
     </gazebo>
     <link name="${namespace}${name}_opening" />
-    <!-- bottle opening (without cap) is at 285mm height -->
+    <!-- bottle opening (without cap) is at 284mm height -->
     <joint name="${namespace}${name}_opening_joint" type="fixed">
       <parent link="${namespace}${name}" />
       <child link="${namespace}${name}_opening" />
-      <origin xyz="0 0 0.285" rpy="0 0 0" />
+      <origin xyz="0 0 0.284" rpy="0 0 0" />
     </joint>
   </xacro:macro>

File: urdf/easy_grasp_bottle.xacro (robot description, xacro)
@@ -32,7 +32,7 @@
       <collision>
         <!-- Schweppes 1-liter plastic bottle -->
-        <origin xyz="0 0 ${0.5*0.25}" rpy="0 0 0" />
+        <origin xyz="0 0 ${0.5*0.284}" rpy="0 0 0" />
         <geometry>
-          <cylinder radius="0.04" length="0.3" />
+          <cylinder radius="0.04" length="0.284" />
         </geometry>
       </collision>
@@ -58,9 +58,9 @@
     </gazebo>
     <link name="${namespace}${name}_opening" />
-    <!-- Schweppes bottle has opening at height 285 mm -->
+    <!-- Schweppes bottle has opening at height 284 mm -->
     <joint name="${namespace}${name}_opening_joint" type="fixed">
       <parent link="${namespace}${name}" />
       <child link="${namespace}${name}_opening" />
-      <origin xyz="0 0 0.285" rpy="0 0 0" />
+      <origin xyz="0 0 0.284" rpy="0 0 0" />
     </joint>
   </xacro:macro>
