Commit message: Rename tiago_world to tiago_barkeeper_world
The package was renamed. All references to the tiago_world package
were updated to the new name as well.

Add walls to the bar.
Add scale parameter to the bar and scale the bar further down.
Otherwise it is too large for the tiago.

File: tiago_barkeeper_world/robots/orange_bottle.xacro (robot description, xacro)
@@ -4,9 +4,9 @@
        xmlns:interface="http://playerstage.sourceforge.net/gazebo/xmlschema/#interface"
        xmlns:xacro="http://www.ros.org/wiki/xacro"
-       name="red_bottle">
-   <xacro:include filename="$(find tiago_world)/urdf/materials.xacro" />
-   <xacro:include filename="$(find tiago_world)/urdf/easy_grasp_bottle.xacro" />
+       name="orange_bottle">
+   <xacro:include filename="$(find tiago_barkeeper_world)/urdf/materials.xacro" />
+   <xacro:include filename="$(find tiago_barkeeper_world)/urdf/easy_grasp_bottle.xacro" />
    <xacro:easy_grasp_bottle
-          namespace="" name="red_bottle" weight="0.2"
-          rvizMaterial="red" gazeboMaterial="Gazebo/Red" />
+          namespace="" name="orange_bottle" weight="0.2"
+          rvizMaterial="orange" gazeboMaterial="Gazebo/Orange" />
 </robot>

File: tiago_barkeeper_world/robots/red_bottle.xacro (robot description, xacro)
@@ -4,9 +4,9 @@
        xmlns:interface="http://playerstage.sourceforge.net/gazebo/xmlschema/#interface"
        xmlns:xacro="http://www.ros.org/wiki/xacro"
-       name="yellow_bottle">
-   <xacro:include filename="$(find tiago_world)/urdf/materials.xacro" />
-   <xacro:include filename="$(find tiago_world)/urdf/easy_grasp_bottle.xacro" />
+       name="red_bottle">
+   <xacro:include filename="$(find tiago_barkeeper_world)/urdf/materials.xacro" />
+   <xacro:include filename="$(find tiago_barkeeper_world)/urdf/easy_grasp_bottle.xacro" />
    <xacro:easy_grasp_bottle
-          namespace="" name="yellow_bottle" weight="0.2"
-          rvizMaterial="yellow" gazeboMaterial="Gazebo/Yellow" />
+          namespace="" name="red_bottle" weight="0.2"
+          rvizMaterial="red" gazeboMaterial="Gazebo/Red" />
 </robot>

File: tiago_barkeeper_world/robots/yellow_bottle.xacro (robot description, xacro)
@@ -4,9 +4,9 @@
        xmlns:interface="http://playerstage.sourceforge.net/gazebo/xmlschema/#interface"
        xmlns:xacro="http://www.ros.org/wiki/xacro"
-       name="orange_bottle">
-   <xacro:include filename="$(find tiago_world)/urdf/materials.xacro" />
-   <xacro:include filename="$(find tiago_world)/urdf/easy_grasp_bottle.xacro" />
+       name="yellow_bottle">
+   <xacro:include filename="$(find tiago_barkeeper_world)/urdf/materials.xacro" />
+   <xacro:include filename="$(find tiago_barkeeper_world)/urdf/easy_grasp_bottle.xacro" />
    <xacro:easy_grasp_bottle
-          namespace="" name="orange_bottle" weight="0.2"
-          rvizMaterial="orange" gazeboMaterial="Gazebo/Orange" />
+          namespace="" name="yellow_bottle" weight="0.2"
+          rvizMaterial="yellow" gazeboMaterial="Gazebo/Yellow" />
 </robot>

File: tiago_barkeeper_world/robots/yellow_glass.xacro (robot description, xacro)
@@ -5,6 +5,6 @@
        xmlns:xacro="http://www.ros.org/wiki/xacro"
        name="yellow_glass">
-   <xacro:include filename="$(find tiago_world)/urdf/materials.xacro" />
-   <xacro:include filename="$(find tiago_world)/urdf/ikea_glass.xacro" />
+   <xacro:include filename="$(find tiago_barkeeper_world)/urdf/materials.xacro" />
+   <xacro:include filename="$(find tiago_barkeeper_world)/urdf/ikea_glass.xacro" />
    <xacro:ikea_glass
           namespace="" name="yellow_glass" liquid_weight="0.1"

File: tiago_barkeeper_world/urdf/apriltag_bottle.xacro (robot description, xacro)
@@ -16,5 +16,5 @@
        (C) 2018 fnh, hendrich@informatik.uni-hamburg.de
        Usage:
-       <xacro:include filename="$(find tiago_world)/urdf/materials.xacro" />
+       <xacro:include filename="$(find tiago_barkeeper_world)/urdf/materials.xacro" />
        <xacro:apriltag_bottle
               namespace="" name="bitter_orange_bottle" weight="1.0"
@@ -22,5 +22,5 @@
               tagFamily="36h11" tagID="201" tagSize="0.06" />
    -->
-  <xacro:include filename="$(find tiago_world)/urdf/bottle.xacro" />
+  <xacro:include filename="$(find tiago_barkeeper_world)/urdf/bottle.xacro" />
   <xacro:include filename="$(find tams_apriltags)/urdf/apriltag_marker.xacro" />
   <xacro:macro name="apriltag_bottle"

File: tiago_barkeeper_world/urdf/bar_counter.xacro (robot description, xacro)
@@ -4,19 +4,21 @@
        xmlns:interface="http://playerstage.sourceforge.net/gazebo/xmlschema/#interface"
        xmlns:xacro="http://www.ros.org/wiki/xacro"
-       name="bar_stool">
-  <!-- ROS xacro/urdf model of a bar stool ("Hocker") with
-       silver/red-velvet texture.
+       name="bar_counter">
+  <!-- ROS xacro/urdf model of a bar counter ("Tresen") with wood
+       texture and some shelves on the back (robot) side.
        Origin is at the bottom, centered in x and y.
        2018.05.17 - created
        (C) 2018 fnh, hendrich@informatik.uni-hamburg.de
        Usage:
-       <xacro:include filename="$(find tiago_world)/urdf/materials.xacro" />
-       <xacro:bar_stool name="stool_1" />
+       <xacro:include filename="$(find tiago_barkeeper_world)/urdf/materials.xacro" />
+       <xacro:bar_counter name="counter" />
    -->
-  <xacro:macro name="bar_stool" params="name" >
+  <xacro:macro name="scale" value="0.00075"/>
+  <xacro:macro name="bar_counter"
+               params="name" >
     <!-- main body with mesh collision and visual model -->
     <link name="${name}">
       <inertial>
-        <mass value="20" />
+        <mass value="200" />
         <origin xyz="0 0 0" rpy="0 0 0" />
         <inertia ixx="0.01" ixy="0" ixz="0" iyy="0.01" iyz="0" izz="0.01" />
@@ -25,5 +27,5 @@
         <origin xyz="0 0 0" rpy="0 0 0" />
         <geometry>
-          <mesh filename="file://$(find tiago_world)/meshes/bar_stool_binary.stl" scale="0.001 0.001 0.001" />
+          <mesh filename="file://$(find tiago_barkeeper_world)/meshes/bartresen_binary.stl" scale="${scale} ${scale} ${scale}" />
         </geometry>
       </collision>
@@ -31,8 +33,8 @@
         <origin xyz="0 0 0" rpy="0 0 0" />
         <geometry>
-          <mesh filename="file://$(find tiago_world)/meshes/bar_stool_binary.stl" scale="0.001 0.001 0.001" />
+          <mesh filename="file://$(find tiago_barkeeper_world)/meshes/bartresen_binary.stl" scale="${scale} ${scale} ${scale}" />
         </geometry>
-        <material name="${name}_bar_stool_gray" >
-          <color rgba="0.7 0.4 0.4 1.0" />
+        <material name="noyer_wood" >
+          <!-- <color rgba="1.0 1.0 1.0 1.0"/> -->
         </material>
       </visual>
@@ -40,5 +42,5 @@
     <gazebo reference="${name}">
       <!-- material/texture definition for Gazebo -->
-      <material>tiago/Coke</material>
+      <material>tiago/Wood</material> -->
       <turnGravityOff>false</turnGravityOff>
       <selfCollide>false</selfCollide>

File: tiago_barkeeper_world/urdf/bar_cupboard.xacro (robot description, xacro)
@@ -4,20 +4,21 @@
        xmlns:interface="http://playerstage.sourceforge.net/gazebo/xmlschema/#interface"
        xmlns:xacro="http://www.ros.org/wiki/xacro"
-       name="bar_counter">
-  <!-- ROS xacro/urdf model of a bar counter ("Tresen") with wood
-       texture and some shelves on the back (robot) side.
+       name="bar_cupboard">
+  <!-- ROS xacro/urdf model of a bar shelf/cupboard with wood
+       texture.
        Origin is at the bottom, centered in x and y.
        2018.05.17 - created
        (C) 2018 fnh, hendrich@informatik.uni-hamburg.de
        Usage:
-       <xacro:include filename="$(find tiago_world)/urdf/materials.xacro" />
-       <xacro:bar_counter name="counter" />
+       <xacro:include filename="$(find tiago_barkeeper_world)/urdf/materials.xacro" />
+       <xacro:bar_cupboard name="cupboard" />
    -->
-  <xacro:macro name="bar_counter"
+  <xacro:property name="scale" value="0.00075" />
+  <xacro:macro name="bar_cupboard"
                params="name" >
     <!-- main body with mesh collision and visual model -->
     <link name="${name}">
       <inertial>
-        <mass value="200" />
+        <mass value="300" />
         <origin xyz="0 0 0" rpy="0 0 0" />
         <inertia ixx="0.01" ixy="0" ixz="0" iyy="0.01" iyz="0" izz="0.01" />
@@ -26,5 +27,5 @@
         <origin xyz="0 0 0" rpy="0 0 0" />
         <geometry>
-          <mesh filename="file://$(find tiago_world)/meshes/bartresen_binary.stl" scale="0.001 0.001 0.001" />
+          <mesh filename="file://$(find tiago_barkeeper_world)/meshes/cupboard_binary.stl" scale="${scale} ${scale} ${scale}" />
         </geometry>
       </collision>
@@ -32,5 +33,5 @@
         <origin xyz="0 0 0" rpy="0 0 0" />
         <geometry>
-          <mesh filename="file://$(find tiago_world)/meshes/bartresen_binary.stl" scale="0.001 0.001 0.001" />
+          <mesh filename="file://$(find tiago_barkeeper_world)/meshes/cupboard_binary.stl" scale="${scale} ${scale} ${scale}" />
         </geometry>
         <material name="noyer_wood" >

File: tiago_barkeeper_world/urdf/bar_demo.xacro (robot description, xacro)
@@ -9,14 +9,12 @@
        Note: no bottles/glasses here, as they need to be spawned later.
   -->
-  <xacro:include filename="$(find tiago_world)/urdf/materials.xacro" />
-  <xacro:include filename="$(find tiago_world)/urdf/bar_counter.xacro" />
-  <xacro:include filename="$(find tiago_world)/urdf/bar_stool.xacro" />
-  <xacro:include filename="$(find tiago_world)/urdf/bar_cupboard.xacro" />
+  <xacro:include filename="$(find tiago_barkeeper_world)/urdf/materials.xacro" />
+  <xacro:include filename="$(find tiago_barkeeper_world)/urdf/bar_counter.xacro" />
+  <xacro:include filename="$(find tiago_barkeeper_world)/urdf/bar_stool.xacro" />
+  <xacro:include filename="$(find tiago_barkeeper_world)/urdf/bar_cupboard.xacro" />
+  <xacro:include filename="$(find tiago_barkeeper_world)/urdf/bar_corner.xacro" />
   <link name="world" />
   <link name="tiago/world" />
-  <joint name="hugo" type="fixed">
-    <parent link="world" />
-    <child  link="tiago/world" />
-  </joint>
+  <xacro:bar_corner />
   <xacro:bar_counter name="counter" />
   <xacro:bar_cupboard name="cupboard" />
@@ -24,4 +22,28 @@
   <xacro:bar_stool name="stool_2" />
   <xacro:bar_stool name="stool_3" />
+  <joint name="world_wall_back_joint" type="fixed">
+    <parent link="world"/>
+    <child link="wall_back"/>
+    <origin xyz="4.12 0.0 0.0" rpy="0 0 0" />
+  </joint>
+  <joint name="world_wall_front_joint" type="fixed">
+    <parent link="world"/>
+    <child link="wall_front"/>
+    <origin xyz="-3.0 0.0 0.0" rpy="0 0 0" />
+  </joint>
+  <joint name="world_wall_left_joint" type="fixed">
+    <parent link="world"/>
+    <child link="wall_left"/>
+    <origin xyz="0.5 3.0 0.0" rpy="0 0 1.5708" />
+  </joint>
+  <joint name="world_wall_right_joint" type="fixed">
+    <parent link="world"/>
+    <child link="wall_right"/>
+    <origin xyz="0.5 -2.88 0.0" rpy="0 0 1.5708" />
+  </joint>
+  <joint name="hugo" type="fixed">
+    <parent link="world" />
+    <child  link="tiago/world" />
+  </joint>
   <joint name="bar_counter_joint" type="fixed">
     <parent link="world" />

File: tiago_barkeeper_world/urdf/bar_stool.xacro (robot description, xacro)
@@ -4,20 +4,20 @@
        xmlns:interface="http://playerstage.sourceforge.net/gazebo/xmlschema/#interface"
        xmlns:xacro="http://www.ros.org/wiki/xacro"
-       name="bar_cupboard">
-  <!-- ROS xacro/urdf model of a bar shelf/cupboard with wood
-       texture.
+       name="bar_stool">
+  <!-- ROS xacro/urdf model of a bar stool ("Hocker") with
+       silver/red-velvet texture.
        Origin is at the bottom, centered in x and y.
        2018.05.17 - created
        (C) 2018 fnh, hendrich@informatik.uni-hamburg.de
        Usage:
-       <xacro:include filename="$(find tiago_world)/urdf/materials.xacro" />
-       <xacro:bar_cupboard name="cupboard" />
+       <xacro:include filename="$(find tiago_barkeeper_world)/urdf/materials.xacro" />
+       <xacro:bar_stool name="stool_1" />
    -->
-  <xacro:macro name="bar_cupboard"
-               params="name" >
+  <xacro:macro name="scale" value="0.00075"/>
+  <xacro:macro name="bar_stool" params="name" >
     <!-- main body with mesh collision and visual model -->
     <link name="${name}">
       <inertial>
-        <mass value="300" />
+        <mass value="20" />
         <origin xyz="0 0 0" rpy="0 0 0" />
         <inertia ixx="0.01" ixy="0" ixz="0" iyy="0.01" iyz="0" izz="0.01" />
@@ -26,5 +26,5 @@
         <origin xyz="0 0 0" rpy="0 0 0" />
         <geometry>
-          <mesh filename="file://$(find tiago_world)/meshes/cupboard_binary.stl" scale="0.001 0.001 0.001" />
+          <mesh filename="file://$(find tiago_barkeeper_world)/meshes/bar_stool_binary.stl" scale="${scale} ${scale} ${scale}" />
         </geometry>
       </collision>
@@ -32,8 +32,8 @@
         <origin xyz="0 0 0" rpy="0 0 0" />
         <geometry>
-          <mesh filename="file://$(find tiago_world)/meshes/cupboard_binary.stl" scale="0.001 0.001 0.001" />
+          <mesh filename="file://$(find tiago_barkeeper_world)/meshes/bar_stool_binary.stl" scale="${scale} ${scale} ${scale}" />
         </geometry>
-        <material name="noyer_wood" >
-          <!-- <color rgba="1.0 1.0 1.0 1.0"/> -->
+        <material name="${name}_bar_stool_gray" >
+          <color rgba="0.7 0.4 0.4 1.0" />
         </material>
       </visual>
@@ -41,5 +41,5 @@
     <gazebo reference="${name}">
       <!-- material/texture definition for Gazebo -->
-      <material>tiago/Wood</material> -->
+      <material>tiago/Coke</material>
       <turnGravityOff>false</turnGravityOff>
       <selfCollide>false</selfCollide>

File: tiago_barkeeper_world/urdf/bottle.xacro (robot description, xacro)
@@ -11,5 +11,5 @@
        (C) 2018 fnh, hendrich@informatik.uni-hamburg.de
        Usage:
-       <xacro:include filename="$(find tiago_world)/urdf/materials.xacro" />
+       <xacro:include filename="$(find tiago_barkeeper_world)/urdf/materials.xacro" />
        <xacro:bottle
               namespace="" name="bitter_lemon_bottle" weight="1.0"
@@ -37,5 +37,5 @@
         <origin xyz="0 0 0" rpy="0 0 0" />
         <geometry>
-          <mesh filename="file://$(find tiago_world)/meshes/bottle_binary.stl" scale="0.001 0.001 0.001" />
+          <mesh filename="file://$(find tiago_barkeeper_world)/meshes/bottle_binary.stl" scale="0.001 0.001 0.001" />
         </geometry>
         <material name="${rvizMaterial}" >

File: tiago_barkeeper_world/urdf/bottle_demo.xacro (robot description, xacro)
@@ -5,9 +5,9 @@
        xmlns:xacro="http://www.ros.org/wiki/xacro"
        name="bottle_demo">
-  <xacro:include filename="$(find tiago_world)/urdf/materials.xacro" />
-  <xacro:include filename="$(find tiago_world)/urdf/bottle.xacro" />
-  <xacro:include filename="$(find tiago_world)/urdf/apriltag_bottle.xacro" />
-  <xacro:include filename="$(find tiago_world)/urdf/easy_grasp_bottle.xacro" />
-  <xacro:include filename="$(find tiago_world)/urdf/ikea_glass.xacro" />
+  <xacro:include filename="$(find tiago_barkeeper_world)/urdf/materials.xacro" />
+  <xacro:include filename="$(find tiago_barkeeper_world)/urdf/bottle.xacro" />
+  <xacro:include filename="$(find tiago_barkeeper_world)/urdf/apriltag_bottle.xacro" />
+  <xacro:include filename="$(find tiago_barkeeper_world)/urdf/easy_grasp_bottle.xacro" />
+  <xacro:include filename="$(find tiago_barkeeper_world)/urdf/ikea_glass.xacro" />
   <link name="world" />
   <link name="tiago/world" />

File: tiago_barkeeper_world/urdf/easy_grasp_bottle.xacro (robot description, xacro)
@@ -4,33 +4,35 @@
        xmlns:interface="http://playerstage.sourceforge.net/gazebo/xmlschema/#interface"
        xmlns:xacro="http://www.ros.org/wiki/xacro"
-       name="ikea_glass">
-  <!-- ROS xacro/urdf model of a standard Ikea glass.
-       For convenience, the origin of the glass is at the bottom;
-       we also create an (empty) link at the center of the opening.
+       name="easy_grasp_bottle">
+  <!-- ROS xacro/urdf model of a (Schweppes) 1-liter plastic bottle.
+       This version adds an extra ring at roughly 2/3 height, to make
+       the bottle more graspable in Gazebo.
+       The origin of the bottle is at the bottom; additionally
+       we also create an (empty) link for the bottle opening.
        2018.05.17 - created
        (C) 2018 fnh, hendrich@informatik.uni-hamburg.de
        Usage:
-       <xacro:include filename="$(find tiago_world)/urdf/materials.xacro" />
-       <xacro:ikea_glass
-              namespace="" name="ikea_glass_1" weight="0.2"
-              rvizMaterial="white" gazeboMaterial="Gazebo/White" />
+       <xacro:include filename="$(find tiago_barkeeper_world)/urdf/materials.xacro" />
+       <xacro:easy_grasp_bottle
+              namespace="" name="easy_grasp__bottle" weight="1.0"
+              rvizMaterial="orange" gazeboMaterial="Gazebo/Orange"
+              tagFamily="36h11" tagID="201" tagSize="0.06" />
    -->
-  <xacro:macro name="ikea_glass"
-               params="namespace name liquid_weight rvizMaterial gazeboMaterial" >
-    <!-- glass main body, mesh used for both collision and visual -->
+  <xacro:macro name="easy_grasp_bottle"
+               params="namespace name weight rvizMaterial gazeboMaterial" >
+    <!-- main body with cylinder collision model and bottle mesh for visual -->
     <link name="${namespace}${name}">
       <inertial>
-        <!-- center of mass is centered in x and y, and in z is approximated
-             by one third of the glass height multiplied by amount of liquid
-             in the glass ... -->
-        <mass value="${0.2+liquid_weight}" />
-        <origin xyz="0 0 ${0.3*0.12*(liquid_weight/0.2)}" rpy="0 0 0" />
+        <!-- center of mass is centered in x and y, and in z is half
+             of the bottle height by amount of liquid in the bottle ... -->
+        <mass value="${weight}" />
+        <origin xyz="0 0 ${0.5*0.25*weight}" rpy="0 0 0" />
         <inertia ixx="0.01" ixy="0" ixz="0" iyy="0.01" iyz="0" izz="0.01" />
       </inertial>
       <collision>
-        <!-- standard IKEA drinking glass, 120mm, upper diam 86, bottom diam 56 -->
-        <origin xyz="0 0 0" rpy="0 0 0" />
+        <!-- Schweppes 1-liter plastic bottle -->
+        <origin xyz="0 0 ${0.5*0.284}" rpy="0 0 0" />
         <geometry>
-          <mesh filename="file://$(find tiago_world)/meshes/ikea_glass_binary.stl" scale="0.001 0.001 0.001" />
+          <cylinder radius="0.04" length="0.284" />
         </geometry>
       </collision>
@@ -38,5 +40,5 @@
         <origin xyz="0 0 0" rpy="0 0 0" />
         <geometry>
-          <mesh filename="file://$(find tiago_world)/meshes/ikea_glass_binary.stl" scale="0.001 0.001 0.001" />
+          <mesh filename="file://$(find tiago_barkeeper_world)/meshes/easy_grasp_bottle_binary.stl" scale="0.001 0.001 0.001" />
         </geometry>
         <material name="${rvizMaterial}" >
@@ -56,8 +58,9 @@
     </gazebo>
     <link name="${namespace}${name}_opening" />
+    <!-- Schweppes bottle has opening at height 284 mm -->
     <joint name="${namespace}${name}_opening_joint" type="fixed">
       <parent link="${namespace}${name}" />
       <child link="${namespace}${name}_opening" />
-      <origin xyz="0 0 0.12" rpy="0 0 0" />
+      <origin xyz="0 0 0.284" rpy="0 0 0" />
     </joint>
   </xacro:macro>
