Commit message: Rename tiago_world to tiago_barkeeper_world
The package was renamed. All references to the tiago_world package
were updated to the new name as well.

Add walls to the bar.
Add scale parameter to the bar and scale the bar further down.
Otherwise it is too large for the tiago.

File: tiago_barkeeper_world/urdf/ikea_glass.xacro (robot description, xacro)
@@ -4,35 +4,33 @@
        xmlns:interface="http://playerstage.sourceforge.net/gazebo/xmlschema/#interface"
        xmlns:xacro="http://www.ros.org/wiki/xacro"
-       name="easy_grasp_bottle">
-  <!-- ROS xacro/urdf model of a (Schweppes) 1-liter plastic bottle.
-       This version adds an extra ring at roughly 2/3 height, to make
-       the bottle more graspable in Gazebo.
-       The origin of the bottle is at the bottom; additionally
-       we also create an (empty) link for the bottle opening.
+       name="ikea_glass">
+  <!-- ROS xacro/urdf model of a standard Ikea glass.
+       For convenience, the origin of the glass is at the bottom;
+       we also create an (empty) link at the center of the opening.
        2018.05.17 - created
        (C) 2018 fnh, hendrich@informatik.uni-hamburg.de
        Usage:
-       <xacro:include filename="$(find tiago_world)/urdf/materials.xacro" />
-       <xacro:easy_grasp_bottle
-              namespace="" name="easy_grasp__bottle" weight="1.0"
-              rvizMaterial="orange" gazeboMaterial="Gazebo/Orange"
-              tagFamily="36h11" tagID="201" tagSize="0.06" />
+       <xacro:include filename="$(find tiago_barkeeper_world)/urdf/materials.xacro" />
+       <xacro:ikea_glass
+              namespace="" name="ikea_glass_1" weight="0.2"
+              rvizMaterial="white" gazeboMaterial="Gazebo/White" />
    -->
-  <xacro:macro name="easy_grasp_bottle"
-               params="namespace name weight rvizMaterial gazeboMaterial" >
-    <!-- main body with cylinder collision model and bottle mesh for visual -->
+  <xacro:macro name="ikea_glass"
+               params="namespace name liquid_weight rvizMaterial gazeboMaterial" >
+    <!-- glass main body, mesh used for both collision and visual -->
     <link name="${namespace}${name}">
       <inertial>
-        <!-- center of mass is centered in x and y, and in z is half
-             of the bottle height by amount of liquid in the bottle ... -->
-        <mass value="${weight}" />
-        <origin xyz="0 0 ${0.5*0.25*weight}" rpy="0 0 0" />
+        <!-- center of mass is centered in x and y, and in z is approximated
+             by one third of the glass height multiplied by amount of liquid
+             in the glass ... -->
+        <mass value="${0.2+liquid_weight}" />
+        <origin xyz="0 0 ${0.3*0.12*(liquid_weight/0.2)}" rpy="0 0 0" />
         <inertia ixx="0.01" ixy="0" ixz="0" iyy="0.01" iyz="0" izz="0.01" />
       </inertial>
       <collision>
-        <!-- Schweppes 1-liter plastic bottle -->
-        <origin xyz="0 0 ${0.5*0.284}" rpy="0 0 0" />
+        <!-- standard IKEA drinking glass, 120mm, upper diam 86, bottom diam 56 -->
+        <origin xyz="0 0 0" rpy="0 0 0" />
         <geometry>
-          <cylinder radius="0.04" length="0.284" />
+          <mesh filename="file://$(find tiago_barkeeper_world)/meshes/ikea_glass_binary.stl" scale="0.001 0.001 0.001" />
         </geometry>
       </collision>
@@ -40,5 +38,5 @@
         <origin xyz="0 0 0" rpy="0 0 0" />
         <geometry>
-          <mesh filename="file://$(find tiago_world)/meshes/easy_grasp_bottle_binary.stl" scale="0.001 0.001 0.001" />
+          <mesh filename="file://$(find tiago_barkeeper_world)/meshes/ikea_glass_binary.stl" scale="0.001 0.001 0.001" />
         </geometry>
         <material name="${rvizMaterial}" >
@@ -58,9 +56,8 @@
     </gazebo>
     <link name="${namespace}${name}_opening" />
-    <!-- Schweppes bottle has opening at height 284 mm -->
     <joint name="${namespace}${name}_opening_joint" type="fixed">
       <parent link="${namespace}${name}" />
       <child link="${namespace}${name}_opening" />
-      <origin xyz="0 0 0.284" rpy="0 0 0" />
+      <origin xyz="0 0 0.12" rpy="0 0 0" />
     </joint>
   </xacro:macro>

File: tiago_barkeeper_world/urdf/tiago_cards_demo.xacro (robot description, xacro)
@@ -5,5 +5,5 @@
        xmlns:xacro="http://www.ros.org/wiki/xacro"
        name="apriltag_demo">
-  <xacro:include filename="$(find tiago_world)/urdf/tiago_command_card.xacro" />
+  <xacro:include filename="$(find tiago_barkeeper_world)/urdf/tiago_command_card.xacro" />
   <xacro:include filename="$(find tams_apriltags)/urdf/apriltag_marker.xacro" />
   <link name="world" />
