Commit message: bottles with labels

File: tiago_barkeeper_world/robots/bottle_coke.xacro (robot description, xacro)
@@ -1,4 +1,4 @@
-<robot name="test_bottle">
-    <link name="test_bottle">
+<robot name="bottle_coke">
+    <link name="bottle_coke">
         <inertial>
             <origin xyz="0 0 0" rpy="0 0 0"/>
@@ -9,5 +9,5 @@
             <origin xyz="0 0 0" rpy="0 0 0"/>
             <geometry>
-                <mesh filename="package://tiago_barkeeper_world/meshes/test_bottle.dae"/>
+                <mesh filename="package://tiago_barkeeper_world/meshes/bottle_coke.dae"/>
             </geometry>
         </visual>
@@ -15,9 +15,9 @@
             <origin xyz="0 0 0" rpy="0 0 0"/>
             <geometry>
-                <mesh filename="package://tiago_barkeeper_world/meshes/test_bottle.dae"/>
+                <mesh filename="package://tiago_barkeeper_world/meshes/bottle_coke.dae"/>
             </geometry>
         </collision>
     </link>
-    <gazebo reference="test_bottle">
+    <gazebo reference="bottle_coke">
         <mu1>1.0</mu1>
         <mu2>1.0</mu2>

File: tiago_barkeeper_world/robots/bottle_fanta.xacro (robot description, xacro)
@@ -1,4 +1,4 @@
-<robot name="test_bottle">
-    <link name="test_bottle">
+<robot name="bottle_fanta">
+    <link name="bottle_fanta">
         <inertial>
             <origin xyz="0 0 0" rpy="0 0 0"/>
@@ -9,5 +9,5 @@
             <origin xyz="0 0 0" rpy="0 0 0"/>
             <geometry>
-                <mesh filename="package://tiago_barkeeper_world/meshes/test_bottle.dae"/>
+                <mesh filename="package://tiago_barkeeper_world/meshes/bottle_fanta.dae"/>
             </geometry>
         </visual>
@@ -15,9 +15,9 @@
             <origin xyz="0 0 0" rpy="0 0 0"/>
             <geometry>
-                <mesh filename="package://tiago_barkeeper_world/meshes/test_bottle.dae"/>
+                <mesh filename="package://tiago_barkeeper_world/meshes/bottle_fanta.dae"/>
             </geometry>
         </collision>
     </link>
-    <gazebo reference="test_bottle">
+    <gazebo reference="bottle_fanta">
         <mu1>1.0</mu1>
         <mu2>1.0</mu2>

File: tiago_barkeeper_world/robots/bottle_pepsi.xacro (robot description, xacro)
@@ -1,4 +1,4 @@
-<robot name="test_bottle">
-    <link name="test_bottle">
+<robot name="bottle_pepsi">
+    <link name="bottle_pepsi">
         <inertial>
             <origin xyz="0 0 0" rpy="0 0 0"/>
@@ -9,5 +9,5 @@
             <origin xyz="0 0 0" rpy="0 0 0"/>
             <geometry>
-                <mesh filename="package://tiago_barkeeper_world/meshes/test_bottle.dae"/>
+                <mesh filename="package://tiago_barkeeper_world/meshes/bottle_pepsi.dae"/>
             </geometry>
         </visual>
@@ -15,9 +15,9 @@
             <origin xyz="0 0 0" rpy="0 0 0"/>
             <geometry>
-                <mesh filename="package://tiago_barkeeper_world/meshes/test_bottle.dae"/>
+                <mesh filename="package://tiago_barkeeper_world/meshes/bottle_pepsi.dae"/>
             </geometry>
         </collision>
     </link>
-    <gazebo reference="test_bottle">
+    <gazebo reference="bottle_pepsi">
         <mu1>1.0</mu1>
         <mu2>1.0</mu2>
