Commit message: Reduce wall size

File: tiago_barkeeper_world/urdf/bar_corner.xacro (robot description, xacro)
@@ -17,5 +17,5 @@
     <link name="wall_back">
       <inertial>
-        <origin xyz="-0.06 0.0 1.5" />
+        <origin xyz="-0.06 0.0 0.15" />
         <mass value="2000" />
         <inertia  ixx="0.01" ixy="0" ixz="0" iyy="0.01" iyz="0" izz="0.01" />
@@ -23,13 +23,13 @@
       <visual>
         <material name="white" />
-        <origin xyz="-0.06 0.0 1.5" />
+        <origin xyz="-0.06 0.0 0.15" />
         <geometry>
-          <box size="0.12 6.0 3.0" />
+          <box size="0.12 6.0 0.3" />
         </geometry>
       </visual>
       <collision>
-        <origin xyz="-0.06 0.0 1.5" />
+        <origin xyz="-0.06 0.0 0.15" />
         <geometry>
-          <box size="0.12 6.0 3.0" />
+          <box size="0.12 6.0 0.3" />
         </geometry>
       </collision>
@@ -47,5 +47,5 @@
     <link name="wall_front">
       <inertial>
-        <origin xyz="-0.06 0.0 1.5" />
+        <origin xyz="-0.06 0.0 0.15" />
         <mass value="2000" />
         <inertia  ixx="0.01" ixy="0" ixz="0" iyy="0.01" iyz="0" izz="0.01" />
@@ -53,13 +53,13 @@
       <visual>
         <material name="white" />
-        <origin xyz="-0.06 0.0 1.5" />
+        <origin xyz="-0.06 0.0 0.15" />
         <geometry>
-          <box size="0.12 6.0 3.0" />
+          <box size="0.12 6.0 0.3" />
         </geometry>
       </visual>
       <collision>
-        <origin xyz="-0.06 0.0 1.5" />
+        <origin xyz="-0.06 0.0 0.15" />
         <geometry>
-          <box size="0.12 6.0 3.0" />
+          <box size="0.12 6.0 0.3" />
         </geometry>
       </collision>
@@ -77,5 +77,5 @@
     <link name="wall_left">
       <inertial>
-        <origin xyz="-0.06 0.0 1.5" />
+        <origin xyz="-0.06 0.0 0.15" />
         <mass value="2000" />
         <inertia  ixx="0.01" ixy="0" ixz="0" iyy="0.01" iyz="0" izz="0.01" />
@@ -83,13 +83,13 @@
       <visual>
         <material name="white" />
-        <origin xyz="-0.06 0.0 1.5" />
+        <origin xyz="-0.06 0.0 0.15" />
         <geometry>
-          <box size="0.12 7.0 3.0" />
+          <box size="0.12 7.0 0.30" />
         </geometry>
       </visual>
       <collision>
-        <origin xyz="-0.06 0.0 1.5" />
+        <origin xyz="-0.06 0.0 0.15" />
         <geometry>
-          <box size="0.12 7.0 3.0" />
+          <box size="0.12 7.0 0.3" />
         </geometry>
       </collision>
@@ -107,5 +107,5 @@
     <link name="wall_right">
       <inertial>
-        <origin xyz="-0.06 0.0 1.5" />
+        <origin xyz="-0.06 0.0 0.15" />
         <mass value="2000" />
         <inertia  ixx="0.01" ixy="0" ixz="0" iyy="0.01" iyz="0" izz="0.01" />
@@ -113,13 +113,13 @@
       <visual>
         <material name="white" />
-        <origin xyz="-0.06 0.0 1.5" />
+        <origin xyz="-0.06 0.0 0.15" />
         <geometry>
-          <box size="0.12 7.0 3.0" />
+          <box size="0.12 7.0 0.3" />
         </geometry>
       </visual>
       <collision>
-        <origin xyz="-0.06 0.0 1.5" />
+        <origin xyz="-0.06 0.0 0.15" />
         <geometry>
-          <box size="0.12 7.0 3.0" />
+          <box size="0.12 7.0 0.3" />
         </geometry>
       </collision>
