Commit message: Add spawn scripts for Gazebo. Enable gravity for the cards.

File: tiago_bartender_world/urdf/command_card_collada.xacro (robot description, xacro)
@@ -17,5 +17,5 @@
         <mass value="0.01" />
         <origin xyz="0 0 0" rpy="0 0 0" />
-        <inertia ixx="0.01" ixy="0" ixz="0" iyy="0.01" iyz="0" izz="0.01" />
+        <inertia ixx="0.001" ixy="0" ixz="0" iyy="0.001" iyz="0" izz="0.001" />
       </inertial>
       <collision>
@@ -36,5 +36,5 @@
       <!-- material/texture definition for Gazebo -->
       <!-- <material>Gazebo/White</material> -->
-      <turnGravityOff>true</turnGravityOff>
+      <turnGravityOff>false</turnGravityOff>
       <selfCollide>false</selfCollide>
       <mu1>100</mu1>
@@ -55,5 +55,5 @@
     </link>
     <gazebo reference="${namespace}${name}_atag_${tag}">
-      <turnGravityOff>true</turnGravityOff>
+      <turnGravityOff>false</turnGravityOff>
       <selfCollide>false</selfCollide>
     </gazebo>
