Commit message: Add Collada models (bar counter/cupboard/stool) with basic wood textures.

File: tiago_bartender_world/urdf/bar_counter.xacro (robot description, xacro)
@@ -27,5 +27,5 @@
         <origin xyz="0 0 0" rpy="0 0 0" />
         <geometry>
-          <mesh filename="file://$(find tiago_bartender_world)/meshes/bartresen_binary.stl" scale="${scale} ${scale} ${scale}" />
+          <mesh filename="file://$(find tiago_bartender_world)/meshes/bartresen.dae" scale="${scale} ${scale} ${scale}" />
         </geometry>
       </collision>
@@ -33,7 +33,7 @@
         <origin xyz="0 0 0" rpy="0 0 0" />
         <geometry>
-          <mesh filename="file://$(find tiago_bartender_world)/meshes/bartresen_binary.stl" scale="${scale} ${scale} ${scale}" />
+          <mesh filename="file://$(find tiago_bartender_world)/meshes/bartresen.dae" scale="${scale} ${scale} ${scale}" />
         </geometry>
-        <material name="noyer_wood" >
+        <material name="maple_wood" >
           <!-- <color rgba="1.0 1.0 1.0 1.0"/> -->
         </material>
@@ -42,5 +42,5 @@
     <gazebo reference="${name}">
       <!-- material/texture definition for Gazebo -->
-      <material>tiago/Wood</material> -->
+      <!-- <material>tiago/Wood</material> -->
       <turnGravityOff>false</turnGravityOff>
       <selfCollide>false</selfCollide>

File: tiago_bartender_world/urdf/bar_cupboard.xacro (robot description, xacro)
@@ -27,5 +27,5 @@
         <origin xyz="0 0 0" rpy="0 0 0" />
         <geometry>
-          <mesh filename="file://$(find tiago_bartender_world)/meshes/cupboard_binary.stl" scale="${scale} ${scale} ${scale}" />
+          <mesh filename="file://$(find tiago_bartender_world)/meshes/cupboard.dae" scale="${scale} ${scale} ${scale}" />
         </geometry>
       </collision>
@@ -33,7 +33,7 @@
         <origin xyz="0 0 0" rpy="0 0 0" />
         <geometry>
-          <mesh filename="file://$(find tiago_bartender_world)/meshes/cupboard_binary.stl" scale="${scale} ${scale} ${scale}" />
+          <mesh filename="file://$(find tiago_bartender_world)/meshes/cupboard.dae" scale="${scale} ${scale} ${scale}" />
         </geometry>
-        <material name="noyer_wood" >
+        <material name="maple_wood" >
           <!-- <color rgba="1.0 1.0 1.0 1.0"/> -->
         </material>
@@ -42,5 +42,5 @@
     <gazebo reference="${name}">
       <!-- material/texture definition for Gazebo -->
-      <material>tiago/Wood</material> -->
+      <!-- <material>tiago/Wood</material> -->
       <turnGravityOff>false</turnGravityOff>
       <selfCollide>false</selfCollide>

File: tiago_bartender_world/urdf/bar_stool.xacro (robot description, xacro)
@@ -26,5 +26,5 @@
         <origin xyz="0 0 0" rpy="0 0 0" />
         <geometry>
-          <mesh filename="file://$(find tiago_bartender_world)/meshes/bar_stool_binary.stl" scale="${scale} ${scale} ${scale}" />
+          <mesh filename="file://$(find tiago_bartender_world)/meshes/bar_stool.dae" scale="${scale} ${scale} ${scale}" />
         </geometry>
       </collision>
@@ -32,5 +32,5 @@
         <origin xyz="0 0 0" rpy="0 0 0" />
         <geometry>
-          <mesh filename="file://$(find tiago_bartender_world)/meshes/bar_stool_binary.stl" scale="${scale} ${scale} ${scale}" />
+          <mesh filename="file://$(find tiago_bartender_world)/meshes/bar_stool.dae" scale="${scale} ${scale} ${scale}" />
         </geometry>
         <material name="${name}_bar_stool_gray" >
@@ -41,5 +41,5 @@
     <gazebo reference="${name}">
       <!-- material/texture definition for Gazebo -->
-      <material>tiago/Coke</material>
+      <!-- <material>tiago/Coke</material>  -->
       <turnGravityOff>false</turnGravityOff>
       <selfCollide>false</selfCollide>

Commit message: Add 3D models of people and launch scripts.

File: tiago_bartender_world/urdf/bar_counter.xacro (robot description, xacro)
@@ -14,7 +14,6 @@
        <xacro:bar_counter name="counter" />
    -->
-  <xacro:macro name="scale" value="0.00075"/>
   <xacro:macro name="bar_counter"
-               params="name" >
+               params="name scale" >
     <!-- main body with mesh collision and visual model -->
     <link name="${name}">

File: tiago_bartender_world/urdf/bar_demo.xacro (robot description, xacro)
@@ -20,5 +20,5 @@
   <link name="tiago/world" />
   <xacro:bar_corner />
-  <xacro:bar_counter name="counter" />
+  <xacro:bar_counter name="counter" scale="0.00075" />
   <xacro:bar_cupboard name="cupboard" />
   <xacro:bar_stool name="stool_1" />

File: tiago_bartender_world/urdf/bar_stool.xacro (robot description, xacro)
@@ -14,6 +14,6 @@
        <xacro:bar_stool name="stool_1" />
    -->
-  <xacro:macro name="scale" value="0.00075"/>
   <xacro:macro name="bar_stool" params="name" >
+    <xacro:property name="scale" value="0.00075"/>
     <!-- main body with mesh collision and visual model -->
     <link name="${name}">

File: tiago_bartender_world/urdf/woman_pointing.urdf (robot description, URDF)
Before this commit: robot woman_pointing, 1 links, 0 joints
Links:
- link woman_pointing_footprint: geometry collision cylinder length=1.9 radius=0.33; collision origin rpy=0 0 -1.57 xyz=0 0 0
