Commit message: correct path to mesh

File: tiago_bartender_world/urdf/woman_pointing.urdf (robot description, URDF)
Before this commit: robot woman_pointing, 1 links, 0 joints
Links:
- link woman_pointing_footprint: geometry collision cylinder length=1.9 radius=0.33; collision origin rpy=0 0 -1.57 xyz=0 0 0

Commit message: Fix <origin> tag.

File: tiago_bartender_world/urdf/woman_pointing.urdf (robot description, URDF)
Before this commit: robot woman_pointing, 1 links, 0 joints
Links:
- link woman_pointing_footprint: geometry collision cylinder length=1.9 radius=0.33; collision mesh filename=package://tiago_bartender_world/meshes/woman_pointing.dae scale=1.05 1.05 1.05
