Commit message: Scale mesh to useful size.

File: tiago_bartender_world/urdf/man_black_guy.urdf (robot description, URDF)
Before this commit: robot man_black_guy, 2 links, 1 joints
Links:
- link man_black_guy/base_footprint: geometry collision cylinder length=0.001 radius=0.30
- link man_black_guy/base_link: geometry collision mesh filename=package://tiago_bartender_world/meshes/man_black_guy.dae scale=0.0014 0.0014 0.0014; visual mesh filename=package://tiago_bartender_world/meshes/man_black_guy.dae scale=0.0014 0.0014 0.0014
Joints:
- joint man_black_guy/base_link_joint: origin xyz=0 0 0.9 rpy=0 0 0 -> xyz=0 0 0.0 rpy=0 0 0
